File: Flight-Controller-PCB/Flight-Controller-PCB.kicad_pcb (KiCad board)
At the start: 2 copper layers, 50 x 50 mm, 78 parts, among them J1 ESC_1, J2 Receiver, J3 ESC_2, J4 ICSP, J5 ESC_3, J6 Aux, J7 ESC_4, J8 Power_In, J9 USB_B_Micro, Q1 BSS138, Q2 BSS138, Q3 PMV48XP,215, Q4 PMV48XP,215, SW1 Push-Switch, U1 MCP6001U, U2 ICM-20689, U3 ATmega32U4-AU, U4 LM1117-5.0, U5 LP2985-3.3, Y1 16MHz, CL 7pF

Commit message: 18 Traces left
Routing:
- net B_RGB_LED: track 0.00 -> 53.7 mm, vias 0 -> 2
- net D7: track 0.00 -> 48.0 mm, vias 0 -> 2
- net A4: track 0.00 -> 42.4 mm, vias 0 -> 2
- net D12: track 0.00 -> 40.5 mm, vias 0 -> 2
- net D16-MOSI: track 7.78 -> 42.4 mm, vias 0 -> 1
- net D15-SCK: track 4.80 -> 39.3 mm, vias 0 -> 1
- net D14-MISO: track 4.81 -> 32.3 mm, vias 0 -> 1
- net +5V: track 256.5 -> 282.5 mm, vias 0 -> 2
- net GND: track 4.86 -> 24.0 mm, vias 10 -> 17
- net A3: track 0.00 -> 16.7 mm, vias 0 -> 2
- net Net-(R16-Pad1): track 0.00 -> 11.7 mm, vias 0 -> 2
- net Net-(R15-Pad1): track 0.00 -> 3.73 mm, vias 0 -> 2
- net VBUS: track 24.4 -> 22.8 mm

Commit message: 5 unrouted
Parts:
- moved C11 0.72 mm to (80.0, 129.9)
- moved R17 0.64 mm to (85.2, 136.1)
Routing:
- net A2: track 0.00 -> 121.2 mm, vias 0 -> 2
- net D5: track 0.00 -> 108.0 mm, vias 0 -> 2
- net D9: track 0.00 -> 86.0 mm, vias 0 -> 2
- net D8: track 0.00 -> 81.6 mm, vias 0 -> 2
- net A1: track 0.00 -> 76.5 mm, vias 0 -> 2
- net A5: track 0.00 -> 65.2 mm, vias 0 -> 2
- net D4: track 0.00 -> 56.9 mm, vias 0 -> 2
- net Aux_Digital: track 0.00 -> 40.3 mm, vias 0 -> 2
- net D6: track 0.00 -> 38.4 mm, vias 0 -> 2
- net RESET: track 22.5 -> 60.1 mm, vias 0 -> 2
- net D11: track 0.00 -> 26.8 mm, vias 0 -> 2
- net IMU_SDA_LH: track 22.0 -> 2.01 mm
- net +5V: track 282.5 -> 294.3 mm
- net A4: track 42.4 -> 32.8 mm
- net Net-(R15-Pad1): track 3.73 -> 9.99 mm, vias 2 -> 3
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
Commit message: Silk screen and DRC then done. One Unrouted bug?'
Parts:
- moved R17 0.85 mm to (85.6, 136.9), turned to 0 degrees
Routing:
- net Net-(R15-Pad1): track 9.99 -> 84.9 mm, vias 3 -> 2
- net IMU_SDA_LH: track 2.01 -> 22.4 mm, vias 0 -> 2
- net +5V: track 294.3 -> 288.6 mm
- net A3: track 18.7 -> 21.4 mm, vias 1 -> 2
- net Net-(R17-Pad1): track 2.73 -> 4.13 mm
- net +3V3: track 46.8 -> 45.5 mm, vias 2 -> 1
- net RESET: track 60.1 -> 59.3 mm
- net D11: track 26.8 -> 27.5 mm
- net B_RGB_LED: track 54.4 -> 54.9 mm
- net GND: track 24.9 -> 24.8 mm, vias 20 -> 21

Commit message: Board complete!
Connections:
- J9 pad 4: Net-(J9-Pad4) -> (no net)
- U2 pad 12: Net-(U2-Pad12) -> (no net)
- U2 pad 22: Net-(U2-Pad22) -> (no net)
- U3 pad 20: RX -> (no net)
- U3 pad 21: TX -> (no net)
- U5 pad 4: Net-(U5-Pad4) -> (no net)
Routing:
- net +3V3: track 45.5 -> 46.7 mm, vias 1 -> 2
- net GND: vias 21 -> 35
Other:
- board text added: "+"
- board text added: "-"
- board text added: "A"
- board text added: "D"
- board text added: "ESC1"
- board text added: "ESC2"
- board text added: "ESC3"
- board text added: "ESC4"
- board text added: "V1.0"
- board text added: "x"
- board text added: "y"
- board text added: "z"
